Commit message: a moveit simulation for mz07l

File: urdf/mz07l/urdf/mz07l.urdf (robot description, URDF)
Before this commit: robot mz07l, 7 links, 6 joints
Links:
- added link Tool, mass 0.0303019437346346; collision mesh filename=package://mz07l/meshes/Tool.STL; visual mesh filename=package://mz07l/meshes/Tool.STL
- link Link3: mass 2.92582839280338 -> 2.9258
- link Link5: mass 0.39428 -> 0.394276330704897
- link Link6: mass 0.030302 -> 0.0303019437346346
- link base_link: mass 7.487 -> 7.48699011088476
Joints:
- added joint J7: type fixed, parent Link6, child Tool, origin xyz=0 0 0.073 rpy=0 0 0, axis 0 0 0
- joint J1: limit lower=0 upper=0 effort=0 velocity=0 -> lower=-2.97 upper=2.97 effort=100 velocity=1
- joint J2: limit lower=0 upper=0 effort=0 velocity=0 -> lower=-2.36 upper=1.40 effort=100 velocity=1
- joint J3: limit lower=0 upper=0 effort=0 velocity=0 -> lower=-2.43 upper=4.71 effort=100 velocity=1
- joint J4: limit lower=0 upper=0 effort=0 velocity=0 -> lower=-3.32 upper=3.32 effort=100 velocity=1
- joint J5: limit lower=0 upper=0 effort=0 velocity=0 -> lower=-2.09 upper=2.09 effort=100 velocity=1
- joint J6: limit lower=0 upper=0 effort=0 velocity=0 -> lower=-6.28 upper=6.28 effort=100 velocity=1
