Commit message: a moveit simulation for mz07l

File: mz07l/urdf/mz07l.urdf (robot description, URDF)
Before this commit: robot mz07l, 7 links, 6 joints
Joints:
- joint J1: limit lower=-2.97 upper=2.97 effort=100 velocity=1 -> lower=0 upper=0 effort=0 velocity=0
- joint J2: limit lower=-2.36 upper=1.40 effort=100 velocity=1 -> lower=0 upper=0 effort=0 velocity=0
- joint J3: limit lower=-2.43 upper=4.71 effort=100 velocity=1 -> lower=0 upper=0 effort=0 velocity=0
- joint J4: limit lower=-3.32 upper=3.32 effort=100 velocity=1 -> lower=0 upper=0 effort=0 velocity=0
- joint J5: limit lower=-2.09 upper=2.09 effort=100 velocity=1 -> lower=0 upper=0 effort=0 velocity=0
- joint J6: limit lower=-6.28 upper=6.28 effort=100 velocity=1 -> lower=0 upper=0 effort=0 velocity=0

Commit message: MZ07L simulation in moveit

File: mz07l/urdf/mz07l.urdf (robot description, URDF)
Before this commit: robot mz07l, 8 links, 7 joints
Links:
- removed link Tool
- added link Tools, mass 0.0303019455167; collision mesh filename=package://mz07l/meshes/Tools.STL; visual mesh filename=package://mz07l/meshes/Tools.STL
- added link base, mass 7.48699011088476; collision mesh filename=package://mz07l/meshes/base.STL; visual mesh filename=package://mz07l/meshes/base.STL
- link Link1: mass 4.412 -> 4.4119668882482
- link Link3: mass 2.9258 -> 2.92582891160545
- link Link5: mass 0.394276330704897 -> 0.39428
- link Link6: mass 0.0303019437346346 -> 0.0303019455167
Joints:
- added joint J0: type fixed, parent base_link, child base, origin xyz=0 0 0 rpy=0 0 0, axis 0 0 0
- joint J1: limit lower=-2.97 upper=2.97 effort=100 velocity=1 -> lower=-2.97 upper=2.97 effort=100 velocity=5.24; parent base_link -> base
- joint J2: limit lower=-2.36 upper=1.40 effort=100 velocity=1 -> lower=-2.36 upper=1.40 effort=100 velocity=4.89; origin xyz=0.05549 0 0.15313 rpy=-1.5708 0 0 -> xyz=0.05 0 0.148 rpy=-1.5708 0 0
- joint J3: limit lower=-2.43 upper=4.71 effort=100 velocity=1 -> lower=-1.169 upper=3.316 effort=100 velocity=6.28; origin xyz=-0.043963 -0.40764 0.0005 rpy=0 0 -0.10743 -> xyz=0 -0.41 0 rpy=0 0 0
- joint J4: limit lower=-3.32 upper=3.32 effort=100 velocity=1 -> lower=-3.32 upper=3.32 effort=100 velocity=9.60
- joint J5: limit lower=-2.09 upper=2.09 effort=100 velocity=1 -> lower=-2.09 upper=2.09 effort=100 velocity=9.60
- joint J6: limit lower=-6.28 upper=6.28 effort=100 velocity=1 -> lower=-6.28 upper=6.28 effort=100 velocity=17.5
- joint J7: child Tool -> Tools
